Commit message: feat(robot_description): add front camera + Gazebo camera plugin
Gives camera_link geometry/inertia and adds a libgazebo_ros_camera sensor publishing /camera/image_raw (640x480 rgb8) for the vision node.

File: ros2/src/robot_description/urdf/simple_diffbot.urdf.xacro (robot description, xacro)
@@ -85,6 +85,15 @@
     <origin xyz="-0.11 0 -0.04"/>
   </joint>
-  <!-- sensor mount placeholders (camera / lidar for later milestones) -->
-  <link name="camera_link"/>
+  <!-- front-facing camera -->
+  <link name="camera_link">
+    <visual>
+      <geometry><box size="0.04 0.04 0.03"/></geometry>
+      <material name="black"><color rgba="0.05 0.05 0.05 1.0"/></material>
+    </visual>
+    <collision>
+      <geometry><box size="0.04 0.04 0.03"/></geometry>
+    </collision>
+    <xacro:box_inertia m="0.03" x="0.04" y="0.04" z="0.03"/>
+  </link>
   <joint name="camera_joint" type="fixed">
     <parent link="base_link"/>
@@ -101,4 +110,35 @@
   <gazebo reference="base_link">
     <material>Gazebo/Blue</material>
+  </gazebo>
+  <gazebo reference="camera_link">
+    <sensor type="camera" name="camera">
+      <update_rate>10.0</update_rate>
+      <camera>
+        <horizontal_fov>1.0471975511965976</horizontal_fov>
+        <image>
+          <width>640</width>
+          <height>480</height>
+          <format>R8G8B8</format>
+        </image>
+        <clip>
+          <near>0.05</near>
+          <far>100</far>
+        </clip>
+      </camera>
+      <plugin name="camera_controller" filename="libgazebo_ros_camera.so">
+        <always_on>true</always_on>
+        <update_rate>10.0</update_rate>
+        <camera_name>camera</camera_name>
+        <image_topic_name>image_raw</image_topic_name>
+        <camera_info_topic_name>camera_info</camera_info_topic_name>
+        <frame_name>camera_link</frame_name>
+        <hack_baseline>0.07</hack_baseline>
+        <distortion_k1>0.0</distortion_k1>
+        <distortion_k2>0.0</distortion_k2>
+        <distortion_k3>0.0</distortion_k3>
+        <distortion_t1>0.0</distortion_t1>
+        <distortion_t2>0.0</distortion_t2>
+      </plugin>
+    </sensor>
   </gazebo>
   <gazebo>
